File: Tph_Synth_Featherwing/dac_ac_gen.sch (KiCad schematic (older format))
At the start: 1 part

Commit message: Add parts for DAC
Parts:
- added C?: C_Small, symbol Device:C_Small
- added R? (x2): R_Small, symbol Device:R_Small
- added TP? (x2): TestPoint, symbol Connector:TestPoint
Connections:
- net labels added: +3V3, GND, SCL, SDA, VOUTA, VOUTB, VOUTC, VOUTD
- wire segments 0 -> 14

Commit message: Boost-converter and inverting opamps
Parts:
- added C? (x4): C_Small, symbol Device:C_Small
- C?: value C_Small -> 100n
- R? (x2): value R_Small -> 2.2k
Connections:
- wire segments 14 -> 36
Changed lines of the file:
@@
 P 4380 3030
 F 0 "C?" V 4151 3030 50  0000 C CNN
-F 1 "C_Small" V 4242 3030 50  0000 C CNN
+F 1 "100n" V 4242 3030 50  0000 C CNN
 F 2 "" H 4380 3030 50  0001 C CNN
 F 3 "~" H 4380 3030 50  0001 C CNN
@@
 Wire Wire Line
 	4110 3850 4110 3770
-Text HLabel 4710 3270 2    50   Output ~ 0
+Text HLabel 5540 3265 2    50   Output ~ 0
 VOUTA
-Text HLabel 4710 3370 2    50   Output ~ 0
+Text HLabel 5540 3365 2    50   Output ~ 0
 VOUTB
-Text HLabel 4710 3470 2    50   Output ~ 0
+Text HLabel 5540 3470 2    50   Output ~ 0
 VOUTC
-Text HLabel 4710 3570 2    50   Output ~ 0
+Text HLabel 5540 3565 2    50   Output ~ 0
 VOUTD
 $Bitmap
@@
 P 3075 3135
 F 0 "R?" H 3134 3181 50  0000 L CNN
-F 1 "R_Small" H 3134 3090 50  0000 L CNN
+F 1 "2.2k" H 3134 3090 50  0000 L CNN
 F 2 "" H 3075 3135 50  0001 C CNN
 F 3 "~" H 3075 3135 50  0001 C CNN
@@
 P 2785 3140
 F 0 "R?" H 2844 3186 50  0000 L CNN
-F 1 "R_Small" H 2844 3095 50  0000 L CNN
+F 1 "2.2k" H 2844 3095 50  0000 L CNN
 F 2 "" H 2785 3140 50  0001 C CNN
 F 3 "~" H 2785 3140 50  0001 C CNN
@@
 Wire Wire Line
 	3075 2890 4110 2890
+$Comp
+L Device:C_Small C?
+U 1 1 5DF8058E
+P 4725 3785
+F 0 "C?" H 4817 3831 50  0000 L CNN
+F 1 "C_Small" H 4817 3740 50  0000 L CNN
+F 2 "" H 4725 3785 50  0001 C CNN
+F 3 "~" H 4725 3785 50  0001 C CNN
+	1    4725 3785
+	1    0    0    -1
+$EndComp
+$Comp
+L Device:C_Small C?
+U 1 1 5DF805CE
+P 4870 3785
+F 0 "C?" H 4962 3831 50  0000 L CNN
+F 1 "C_Small" H 4962 3740 50  0000 L CNN
+F 2 "" H 4870 3785 50  0001 C CNN
+F 3 "~" H 4870 3785 50  0001 C CNN
+	1    4870 3785
+	1    0    0    -1
+$EndComp
+$Comp
+L Device:C_Small C?
+U 1 1 5DF805F6
+P 5015 3785
+F 0 "C?" H 5107 3831 50  0000 L CNN
+F 1 "C_Small" H 5107 3740 50  0000 L CNN
+F 2 "" H 5015 3785 50  0001 C CNN
+F 3 "~" H 5015 3785 50  0001 C CNN
+	1    5015 3785
+	1    0    0    -1
+$EndComp
+$Comp
+L Device:C_Small C?
+U 1 1 5DF80626
+P 5165 3785
+F 0 "C?" H 5257 3831 50  0000 L CNN
+F 1 "C_Small" H 5257 3740 50  0000 L CNN
+F 2 "" H 5165 3785 50  0001 C CNN
+F 3 "~" H 5165 3785 50  0001 C CNN
+	1    5165 3785
+	1    0    0    -1
+$EndComp
+Wire Wire Line
+	4710 3270 5165 3270
+Wire Wire Line
+	5540 3270 5540 3265
+Wire Wire Line
+	4710 3370 5015 3370
+Wire Wire Line
+	5540 3370 5540 3365
+Wire Wire Line
+	4710 3470 4870 3470
+Wire Wire Line
+	5540 3570 5540 3565
+Wire Wire Line
+	4725 3685 4725 3570
+Wire Wire Line
+	4710 3570 4725 3570
+Connection ~ 4725 3570
+Wire Wire Line
+	4725 3570 5540 3570
+Wire Wire Line
+	4870 3685 4870 3470
+Connection ~ 4870 3470
+Wire Wire Line
+	4870 3470 5540 3470
+Wire Wire Line
+	5015 3685 5015 3370
+Connection ~ 5015 3370
+Wire Wire Line
+	5015 3370 5540 3370
+Wire Wire Line
+	5165 3685 5165 3270
+Connection ~ 5165 3270
+Wire Wire Line
+	5165 3270 5540 3270
+Wire Wire Line
+	4725 3885 4725 4000
+Wire Wire Line
+	4725 4000 4870 4000
+Wire Wire Line
+	4870 4000 4870 3885
+Wire Wire Line
+	4870 4000 5015 4000
+Wire Wire Line
+	5015 4000 5015 3885
+Connection ~ 4870 4000
+Wire Wire Line
+	5015 4000 5165 4000
+Wire Wire Line
+	5165 4000 5165 3885
+Connection ~ 5015 4000
+$Comp
+L power:GND #PWR?
+U 1 1 5DF82C9C
+P 5165 4000
+F 0 "#PWR?" H 5165 3750 50  0001 C CNN
+F 1 "GND" H 5170 3827 50  0000 C CNN
+F 2 "" H 5165 4000 50  0001 C CNN
+F 3 "" H 5165 4000 50  0001 C CNN
+	1    5165 4000
+	1    0    0    -1
+$EndComp
+Connection ~ 5165 4000
 $EndSCHEMATC

Commit message: Added first-cut of schematic
Parts:
- C14, C15, C16, C17: renamed from C?; value C_Small -> 100n
- gave numbers to parts that had none: 6
Changed lines of the file:
@@
 $EndDescr
 $Comp
-L Analog_DAC:MCP4728 U?
+L Analog_DAC:MCP4728 U4
 U 1 1 5DCBF8FE
 P 4110 3370
-F 0 "U?" H 4110 3848 50  0000 C CNN
+F 0 "U4" H 4110 3848 50  0000 C CNN
 F 1 "MCP4728" H 4110 3757 50  0000 C CNN
 F 2 "Package_SO:MSOP-10_3x3mm_P0.5mm" H 4110 2770 50  0001 C CNN
@@
 $EndComp
 $Comp
-L Device:C_Small C?
+L Device:C_Small C13
 U 1 1 5DECCADB
 P 4380 3030
-F 0 "C?" V 4151 3030 50  0000 C CNN
+F 0 "C13" V 4151 3030 50  0000 C CNN
 F 1 "100n" V 4242 3030 50  0000 C CNN
 F 2 "" H 4380 3030 50  0001 C CNN
@@
 $EndBitmap
 $Comp
-L Device:R_Small R?
+L Device:R_Small R17
 U 1 1 5DECE9C2
 P 3075 3135
-F 0 "R?" H 3134 3181 50  0000 L CNN
+F 0 "R17" H 3134 3181 50  0000 L CNN
 F 1 "2.2k" H 3134 3090 50  0000 L CNN
 F 2 "" H 3075 3135 50  0001 C CNN
@@
 $EndComp
 $Comp
-L Device:R_Small R?
+L Device:R_Small R16
 U 1 1 5DECEA02
 P 2785 3140
-F 0 "R?" H 2844 3186 50  0000 L CNN
+F 0 "R16" H 2844 3186 50  0000 L CNN
 F 1 "2.2k" H 2844 3095 50  0000 L CNN
 F 2 "" H 2785 3140 50  0001 C CNN
@@
 SDA
 $Comp
-L Connector:TestPoint TP?
+L Connector:TestPoint TP6
 U 1 1 5DECF0BD
 P 3510 3470
-F 0 "TP?" V 3705 3544 50  0000 C CNN
+F 0 "TP6" V 3705 3544 50  0000 C CNN
 F 1 "TestPoint" V 3614 3544 50  0000 C CNN
 F 2 "" H 3710 3470 50  0001 C CNN
@@
 $EndComp
 $Comp
-L Connector:TestPoint TP?
+L Connector:TestPoint TP7
 U 1 1 5DECF142
 P 3510 3570
-F 0 "TP?" V 3705 3644 50  0000 C CNN
+F 0 "TP7" V 3705 3644 50  0000 C CNN
 F 1 "TestPoint" V 3614 3644 50  0000 C CNN
 F 2 "" H 3710 3570 50  0001 C CNN
@@
 	3075 2890 4110 2890
 $Comp
-L Device:C_Small C?
+L Device:C_Small C14
 U 1 1 5DF8058E
 P 4725 3785
-F 0 "C?" H 4817 3831 50  0000 L CNN
-F 1 "C_Small" H 4817 3740 50  0000 L CNN
+F 0 "C14" H 4817 3831 50  0000 L CNN
+F 1 "100n" H 4817 3740 50  0000 L CNN
 F 2 "" H 4725 3785 50  0001 C CNN
 F 3 "~" H 4725 3785 50  0001 C CNN
@@
 $EndComp
 $Comp
-L Device:C_Small C?
+L Device:C_Small C15
 U 1 1 5DF805CE
 P 4870 3785
-F 0 "C?" H 4962 3831 50  0000 L CNN
-F 1 "C_Small" H 4962 3740 50  0000 L CNN
+F 0 "C15" H 4962 3831 50  0000 L CNN
+F 1 "100n" H 4962 3740 50  0000 L CNN
 F 2 "" H 4870 3785 50  0001 C CNN
 F 3 "~" H 4870 3785 50  0001 C CNN
@@
 $EndComp
 $Comp
-L Device:C_Small C?
+L Device:C_Small C16
 U 1 1 5DF805F6
 P 5015 3785
-F 0 "C?" H 5107 3831 50  0000 L CNN
-F 1 "C_Small" H 5107 3740 50  0000 L CNN
+F 0 "C16" H 5107 3831 50  0000 L CNN
+F 1 "100n" H 5107 3740 50  0000 L CNN
 F 2 "" H 5015 3785 50  0001 C CNN
 F 3 "~" H 5015 3785 50  0001 C CNN
@@
 $EndComp
 $Comp
-L Device:C_Small C?
+L Device:C_Small C17
 U 1 1 5DF80626
 P 5165 3785
-F 0 "C?" H 5257 3831 50  0000 L CNN
-F 1 "C_Small" H 5257 3740 50  0000 L CNN
+F 0 "C17" H 5257 3831 50  0000 L CNN
+F 1 "100n" H 5257 3740 50  0000 L CNN
 F 2 "" H 5165 3785 50  0001 C CNN
 F 3 "~" H 5165 3785 50  0001 C CNN
@@
 Connection ~ 5015 4000
 $Comp
-L power:GND #PWR?
+L power:GND #PWR019
 U 1 1 5DF82C9C
 P 5165 4000
-F 0 "#PWR?" H 5165 3750 50  0001 C CNN
+F 0 "#PWR019" H 5165 3750 50  0001 C CNN
 F 1 "GND" H 5170 3827 50  0000 C CNN
 F 2 "" H 5165 4000 50  0001 C CNN

Commit message: Initial attempt at PCB
Signed-off-by: Tisham Dhar <whatnickd@gmail.com>
Parts:
- C13, C14, C15, C16, C17: footprint (none) -> Capacitor_SMD:C_0603_1608Metric
- R16, R17: footprint (none) -> Resistor_SMD:R_0603_1608Metric
- TP6, TP7: footprint (none) -> TestPoint:TestPoint_Pad_D1.0mm
Changed lines of the file:
@@
 F 0 "C13" V 4151 3030 50  0000 C CNN
 F 1 "100n" V 4242 3030 50  0000 C CNN
-F 2 "" H 4380 3030 50  0001 C CNN
+F 2 "Capacitor_SMD:C_0603_1608Metric" H 4380 3030 50  0001 C CNN
 F 3 "~" H 4380 3030 50  0001 C CNN
 	1    4380 3030
@@
 F 0 "R17" H 3134 3181 50  0000 L CNN
 F 1 "2.2k" H 3134 3090 50  0000 L CNN
-F 2 "" H 3075 3135 50  0001 C CNN
+F 2 "Resistor_SMD:R_0603_1608Metric" H 3075 3135 50  0001 C CNN
 F 3 "~" H 3075 3135 50  0001 C CNN
 	1    3075 3135
@@
 F 0 "R16" H 2844 3186 50  0000 L CNN
 F 1 "2.2k" H 2844 3095 50  0000 L CNN
-F 2 "" H 2785 3140 50  0001 C CNN
+F 2 "Resistor_SMD:R_0603_1608Metric" H 2785 3140 50  0001 C CNN
 F 3 "~" H 2785 3140 50  0001 C CNN
 	1    2785 3140
@@
 F 0 "TP6" V 3705 3544 50  0000 C CNN
 F 1 "TestPoint" V 3614 3544 50  0000 C CNN
-F 2 "" H 3710 3470 50  0001 C CNN
+F 2 "TestPoint:TestPoint_Pad_D1.0mm" H 3710 3470 50  0001 C CNN
 F 3 "~" H 3710 3470 50  0001 C CNN
 	1    3510 3470
@@
 F 0 "TP7" V 3705 3644 50  0000 C CNN
 F 1 "TestPoint" V 3614 3644 50  0000 C CNN
-F 2 "" H 3710 3570 50  0001 C CNN
+F 2 "TestPoint:TestPoint_Pad_D1.0mm" H 3710 3570 50  0001 C CNN
 F 3 "~" H 3710 3570 50  0001 C CNN
 	1    3510 3570
@@
 F 0 "C14" H 4817 3831 50  0000 L CNN
 F 1 "100n" H 4817 3740 50  0000 L CNN
-F 2 "" H 4725 3785 50  0001 C CNN
+F 2 "Capacitor_SMD:C_0603_1608Metric" H 4725 3785 50  0001 C CNN
 F 3 "~" H 4725 3785 50  0001 C CNN
 	1    4725 3785
@@
 F 0 "C15" H 4962 3831 50  0000 L CNN
 F 1 "100n" H 4962 3740 50  0000 L CNN
-F 2 "" H 4870 3785 50  0001 C CNN
+F 2 "Capacitor_SMD:C_0603_1608Metric" H 4870 3785 50  0001 C CNN
 F 3 "~" H 4870 3785 50  0001 C CNN
 	1    4870 3785
@@
 F 0 "C16" H 5107 3831 50  0000 L CNN
 F 1 "100n" H 5107 3740 50  0000 L CNN
-F 2 "" H 5015 3785 50  0001 C CNN
+F 2 "Capacitor_SMD:C_0603_1608Metric" H 5015 3785 50  0001 C CNN
 F 3 "~" H 5015 3785 50  0001 C CNN
 	1    5015 3785
@@
 F 0 "C17" H 5257 3831 50  0000 L CNN
 F 1 "100n" H 5257 3740 50  0000 L CNN
-F 2 "" H 5165 3785 50  0001 C CNN
+F 2 "Capacitor_SMD:C_0603_1608Metric" H 5165 3785 50  0001 C CNN
 F 3 "~" H 5165 3785 50  0001 C CNN
 	1    5165 3785
