File: Tph_Synth_Featherwing/boost_converter.sch (KiCad schematic (older format))
At the start: 0 parts

Commit message: Progress on sub-sheet labels and boost converter
Parts:
- added C? (x3): C_Small, symbol Device:C_Small
- added L?: L, symbol Device:L
- added R? (x3): R_Small, symbol Device:R_Small
- added U?: PAM2401SCADJ, SOP65P490X110-8N, symbol PAM2401SCADJ:PAM2401SCADJ

Commit message: Boost-converter and inverting opamps
Parts:
- removed R?: R_Small, symbol Device:R_Small
- added D? (x2): D_Schottky, symbol Device:D_Schottky
- added JP?: boost_disable, symbol Jumper:SolderJumper_2_Open
- added R?: 10k, symbol Device:R_Small
- C? (x3): value C_Small -> 22u
- L?: value L -> 2.2uH/3A
- R?: value R_Small -> 100k
- R?: value R_Small -> 750k
Connections:
- net labels added: 5V_OUT, FB, GND, VBAT, VUSB
- wire segments 0 -> 39
Changed lines of the file:
@@
 Data
 89 50 4E 47 0D 0A 1A 0A 00 00 00 0D 49 48 44 52 00 00 02 D6 00 00 01 48 08 02 00 00 00 FB F6 2E
-3F 00 00 00 03 73 42 49 54 08 08 08 DB E1 4F E0 00 00 00 09 70 48 59 73 00 00 12 74 00 00 12 74
-01 DE 66 1F 78 00 00 20 00 49 44 41 54 78 9C EC BD 69 70 1C E7 99 E7 F9 E4 59 55 59 37 EA C2 51
+3F 00 00 00 03 73 42 49 54 08 08 08 DB E1 4F E0 00 00 00 09 70 48 59 73 00 00 12 5C 00 00 12 5C
+01 68 C4 36 89 00 00 20 00 49 44 41 54 78 9C EC BD 69 70 1C E7 99 E7 F9 E4 59 55 59 37 EA C2 51
 40 A1 70 12 00 2F F0 02 41 91 22 25 D9 26 45 59 B6 D9 B6 25 EF B6 A7 27 DA BD 3B E3 EE 88 8E 8D
 D8 D8 88 8E ED F9 E2 89 E8 99 DD FD 32 13 F6 CE EC 7A BB DB 61 AB DB ED B6 2D 89 32 4D B7 25 9A
@@
 P 4080 2720
 F 0 "L?" H 4039 2674 50  0000 R CNN
-F 1 "L" H 4039 2765 50  0000 R CNN
+F 1 "2.2uH/3A" H 4039 2765 50  0000 R CNN
 F 2 "" H 4080 2720 50  0001 C CNN
 F 3 "~" H 4080 2720 50  0001 C CNN
@@
 L Device:C_Small C?
 U 1 1 5DF57921
-P 4080 3210
-F 0 "C?" H 4172 3256 50  0000 L CNN
-F 1 "C_Small" H 4172 3165 50  0000 L CNN
-F 2 "" H 4080 3210 50  0001 C CNN
-F 3 "~" H 4080 3210 50  0001 C CNN
-	1    4080 3210
-	1    0    0    -1
-$EndComp
-$Comp
-L Device:R_Small R?
-U 1 1 5DF57B58
-P 4085 3635
-F 0 "R?" H 4144 3681 50  0000 L CNN
-F 1 "R_Small" H 4144 3590 50  0000 L CNN
-F 2 "" H 4085 3635 50  0001 C CNN
-F 3 "~" H 4085 3635 50  0001 C CNN
-	1    4085 3635
+P 3840 2845
+F 0 "C?" H 3932 2891 50  0000 L CNN
+F 1 "22u" H 3932 2800 50  0000 L CNN
+F 2 "" H 3840 2845 50  0001 C CNN
+F 3 "~" H 3840 2845 50  0001 C CNN
+	1    3840 2845
 	1    0    0    -1
 $EndComp
@@
 P 6490 3320
 F 0 "R?" H 6549 3366 50  0000 L CNN
-F 1 "R_Small" H 6549 3275 50  0000 L CNN
+F 1 "100k" H 6549 3275 50  0000 L CNN
 F 2 "" H 6490 3320 50  0001 C CNN
 F 3 "~" H 6490 3320 50  0001 C CNN
@@
 P 6490 2925
 F 0 "R?" H 6549 2971 50  0000 L CNN
-F 1 "R_Small" H 6549 2880 50  0000 L CNN
+F 1 "750k" H 6549 2880 50  0000 L CNN
 F 2 "" H 6490 2925 50  0001 C CNN
 F 3 "~" H 6490 2925 50  0001 C CNN
@@
 L Device:C_Small C?
 U 1 1 5DF5927E
-P 7140 3200
-F 0 "C?" H 7232 3246 50  0000 L CNN
-F 1 "C_Small" H 7232 3155 50  0000 L CNN
-F 2 "" H 7140 3200 50  0001 C CNN
-F 3 "~" H 7140 3200 50  0001 C CNN
-	1    7140 3200
+P 7140 2915
+F 0 "C?" H 7232 2961 50  0000 L CNN
+F 1 "22u" H 7232 2870 50  0000 L CNN
+F 2 "" H 7140 2915 50  0001 C CNN
+F 3 "~" H 7140 2915 50  0001 C CNN
+	1    7140 2915
 	1    0    0    -1
 $EndComp
@@
 L Device:C_Small C?
 U 1 1 5DF59D11
-P 6745 2920
-F 0 "C?" H 6837 2966 50  0000 L CNN
-F 1 "C_Small" H 6837 2875 50  0000 L CNN
-F 2 "" H 6745 2920 50  0001 C CNN
-F 3 "~" H 6745 2920 50  0001 C CNN
-	1    6745 2920
+P 6905 2915
+F 0 "C?" H 6997 2961 50  0000 L CNN
+F 1 "22u" H 6997 2870 50  0000 L CNN
+F 2 "" H 6905 2915 50  0001 C CNN
+F 3 "~" H 6905 2915 50  0001 C CNN
+	1    6905 2915
 	1    0    0    -1
 $EndComp
+$Comp
+L Device:R_Small R?
+U 1 1 5DF5FAA6
+P 4495 2700
+F 0 "R?" H 4554 2746 50  0000 L CNN
+F 1 "10k" H 4554 2655 50  0000 L CNN
+F 2 "" H 4495 2700 50  0001 C CNN
+F 3 "~" H 4495 2700 50  0001 C CNN
+	1    4495 2700
+	1    0    0    -1
+$EndComp
+Wire Wire Line
+	4905 2645 4685 2645
+Wire Wire Line
+	4685 2645 4685 2600
+Wire Wire Line
+	4685 2600 4495 2600
+Wire Wire Line
+	4270 2600 4270 2570
+Wire Wire Line
+	4080 2570 3840 2570
+Connection ~ 4495 2600
+Wire Wire Line
+	4495 2600 4270 2600
+Wire Wire Line
+	4075 2570 4080 2570
+Connection ~ 4080 2570
+Wire Wire Line
+	4495 2800 4495 2845
+Wire Wire Line
+	4495 2845 4905 2845
+Wire Wire Line
+	4080 2570 4270 2570
+Text HLabel 3705 2570 0    50   Input ~ 0
+VBAT
+Wire Wire Line
+	6305 2645 6490 2645
+Wire Wire Line
+	6490 2645 6490 2825
+Wire Wire Line
+	6490 3220 6490 3025
+Wire Wire Line
+	6305 3645 6490 3645
+Wire Wire Line
+	6305 3745 6490 3745
+Wire Wire Line
+	6490 3420 6490 3645
+Connection ~ 6490 3645
+Wire Wire Line
+	6490 3645 6490 3745
+$Comp
+L power:GND #PWR?
+U 1 1 5DF63EA2
+P 6490 3875
+F 0 "#PWR?" H 6490 3625 50  0001 C CNN
+F 1 "GND" H 6495 3702 50  0000 C CNN
+F 2 "" H 6490 3875 50  0001 C CNN
+F 3 "" H 6490 3875 50  0001 C CNN
+	1    6490 3875
+	1    0    0    -1
+$EndComp
+Wire Wire Line
+	6490 3745 6490 3875
+Connection ~ 6490 3745
+Wire Wire Line
+	6490 2645 6905 2645
+Wire Wire Line
+	7140 2645 7140 2815
+Connection ~ 6490 2645
+Wire Wire Line
+	6905 2645 6905 2815
+Connection ~ 6905 2645
+Wire Wire Line
+	6905 3015 6905 3180
+Wire Wire Line
+	6905 3180 7140 3180
+Wire Wire Line
+	7140 3180 7140 3015
+$Comp
+L power:GND #PWR?
+U 1 1 5DF64C25
+P 7140 3180
+F 0 "#PWR?" H 7140 2930 50  0001 C CNN
+F 1 "GND" H 7145 3007 50  0000 C CNN
+F 2 "" H 7140 3180 50  0001 C CNN
+F 3 "" H 7140 3180 50  0001 C CNN
+	1    7140 3180
+	1    0    0    -1
+$EndComp
+Connection ~ 7140 3180
+Wire Wire Line
+	4905 3045 4785 3045
+Text Label 4785 3045 0    50   ~ 0
+FB
+Text Label 6490 3125 0    50   ~ 0
+FB
+Wire Wire Line
+	4905 3245 4080 3245
+Wire Wire Line
+	4080 3245 4080 2870
+$Comp
+L power:GND #PWR?
+U 1 1 5DF6662F
+P 3840 3100
+F 0 "#PWR?" H 3840 2850 50  0001 C CNN
+F 1 "GND" H 3845 2927 50  0000 C CNN
+F 2 "" H 3840 3100 50  0001 C CNN
+F 3 "" H 3840 3100 50  0001 C CNN
+	1    3840 3100
+	1    0    0    -1
+$EndComp
+Wire Wire Line
+	3840 2745 3840 2570
+Connection ~ 3840 2570
+Wire Wire Line
+	3840 2570 3705 2570
+Wire Wire Line
+	3840 3100 3840 2945
+Wire Wire Line
+	6905 2645 7140 2645
+Connection ~ 7140 2645
+Wire Wire Line
+	7140 2645 7565 2645
+$Comp
+L Device:D_Schottky D?
+U 1 1 5DF67867
+P 7715 2645
+F 0 "D?" H 7715 2429 50  0000 C CNN
+F 1 "D_Schottky" H 7715 2520 50  0000 C CNN
+F 2 "" H 7715 2645 50  0001 C CNN
+F 3 "~" H 7715 2645 50  0001 C CNN
+	1    7715 2645
+	-1   0    0    1
+$EndComp
+Text HLabel 8175 2645 2    50   Output ~ 0
+5V_OUT
+$Comp
+L Jumper:SolderJumper_2_Open JP?
+U 1 1 5DF6A516
+P 4495 2995
+F 0 "JP?" V 4449 3063 50  0000 L CNN
+F 1 "boost_disable" V 4540 3063 50  0000 L CNN
+F 2 "" H 4495 2995 50  0001 C CNN
+F 3 "~" H 4495 2995 50  0001 C CNN
+	1    4495 2995
+	0    1    1    0
+$EndComp
+$Comp
+L power:GND #PWR?
+U 1 1 5DF6A5BE
+P 4495 3425
+F 0 "#PWR?" H 4495 3175 50  0001 C CNN
+F 1 "GND" H 4500 3252 50  0000 C CNN
+F 2 "" H 4495 3425 50  0001 C CNN
+F 3 "" H 4495 3425 50  0001 C CNN
+	1    4495 3425
+	1    0    0    -1
+$EndComp
+Connection ~ 4495 2845
+Wire Wire Line
+	4495 3145 4495 3425
+$Comp
+L Device:D_Schottky D?
+U 1 1 5DF7CB12
+P 7720 2940
+F 0 "D?" H 7720 2724 50  0000 C CNN
+F 1 "D_Schottky" H 7720 2815 50  0000 C CNN
+F 2 "" H 7720 2940 50  0001 C CNN
+F 3 "~" H 7720 2940 50  0001 C CNN
+	1    7720 2940
+	-1   0    0    1
+$EndComp
+Text HLabel 7550 3090 3    50   Input ~ 0
+VUSB
+Wire Wire Line
+	7550 3090 7550 2940
+Wire Wire Line
+	7550 2940 7570 2940
+Wire Wire Line
+	7870 2940 8005 2940
+Wire Wire Line
+	8005 2940 8005 2645
+Wire Wire Line
+	7865 2645 8005 2645
+Connection ~ 8005 2645
+Wire Wire Line
+	8005 2645 8175 2645
 $EndSCHEMATC

Commit message: Added first-cut of schematic
Parts:
- gave numbers to parts that had none: 11
Changed lines of the file:
@@
 $EndBitmap
 $Comp
-L PAM2401SCADJ:PAM2401SCADJ U?
+L PAM2401SCADJ:PAM2401SCADJ U1
 U 1 1 5DF574F0
 P 5605 3245
-F 0 "U?" H 5605 4115 50  0000 C CNN
+F 0 "U1" H 5605 4115 50  0000 C CNN
 F 1 "PAM2401SCADJ" H 5605 4024 50  0000 C CNN
 F 2 "SOP65P490X110-8N" H 5605 3245 50  0001 L BNN
@@
 $EndComp
 $Comp
-L Device:L L?
+L Device:L L1
 U 1 1 5DF576A6
 P 4080 2720
-F 0 "L?" H 4039 2674 50  0000 R CNN
+F 0 "L1" H 4039 2674 50  0000 R CNN
 F 1 "2.2uH/3A" H 4039 2765 50  0000 R CNN
 F 2 "" H 4080 2720 50  0001 C CNN
@@
 $EndComp
 $Comp
-L Device:C_Small C?
+L Device:C_Small C1
 U 1 1 5DF57921
 P 3840 2845
-F 0 "C?" H 3932 2891 50  0000 L CNN
+F 0 "C1" H 3932 2891 50  0000 L CNN
 F 1 "22u" H 3932 2800 50  0000 L CNN
 F 2 "" H 3840 2845 50  0001 C CNN
@@
 $EndComp
 $Comp
-L Device:R_Small R?
+L Device:R_Small R3
 U 1 1 5DF588CE
 P 6490 3320
-F 0 "R?" H 6549 3366 50  0000 L CNN
+F 0 "R3" H 6549 3366 50  0000 L CNN
 F 1 "100k" H 6549 3275 50  0000 L CNN
 F 2 "" H 6490 3320 50  0001 C CNN
@@
 $EndComp
 $Comp
-L Device:R_Small R?
+L Device:R_Small R2
 U 1 1 5DF58910
 P 6490 2925
-F 0 "R?" H 6549 2971 50  0000 L CNN
+F 0 "R2" H 6549 2971 50  0000 L CNN
 F 1 "750k" H 6549 2880 50  0000 L CNN
 F 2 "" H 6490 2925 50  0001 C CNN
@@
 $EndComp
 $Comp
-L Device:C_Small C?
+L Device:C_Small C3
 U 1 1 5DF5927E
 P 7140 2915
-F 0 "C?" H 7232 2961 50  0000 L CNN
+F 0 "C3" H 7232 2961 50  0000 L CNN
 F 1 "22u" H 7232 2870 50  0000 L CNN
 F 2 "" H 7140 2915 50  0001 C CNN
@@
 $EndComp
 $Comp
-L Device:C_Small C?
+L Device:C_Small C2
 U 1 1 5DF59D11
 P 6905 2915
-F 0 "C?" H 6997 2961 50  0000 L CNN
+F 0 "C2" H 6997 2961 50  0000 L CNN
 F 1 "22u" H 6997 2870 50  0000 L CNN
 F 2 "" H 6905 2915 50  0001 C CNN
@@
 $EndComp
 $Comp
-L Device:R_Small R?
+L Device:R_Small R1
 U 1 1 5DF5FAA6
 P 4495 2700
-F 0 "R?" H 4554 2746 50  0000 L CNN
+F 0 "R1" H 4554 2746 50  0000 L CNN
 F 1 "10k" H 4554 2655 50  0000 L CNN
 F 2 "" H 4495 2700 50  0001 C CNN
@@
 	6490 3645 6490 3745
 $Comp
-L power:GND #PWR?
+L power:GND #PWR010
 U 1 1 5DF63EA2
 P 6490 3875
-F 0 "#PWR?" H 6490 3625 50  0001 C CNN
+F 0 "#PWR010" H 6490 3625 50  0001 C CNN
 F 1 "GND" H 6495 3702 50  0000 C CNN
 F 2 "" H 6490 3875 50  0001 C CNN
@@
 	7140 3180 7140 3015
 $Comp
-L power:GND #PWR?
+L power:GND #PWR011
 U 1 1 5DF64C25
 P 7140 3180
-F 0 "#PWR?" H 7140 2930 50  0001 C CNN
+F 0 "#PWR011" H 7140 2930 50  0001 C CNN
 F 1 "GND" H 7145 3007 50  0000 C CNN
 F 2 "" H 7140 3180 50  0001 C CNN
@@
 	4080 3245 4080 2870
 $Comp
-L power:GND #PWR?
+L power:GND #PWR012
 U 1 1 5DF6662F
 P 3840 3100
-F 0 "#PWR?" H 3840 2850 50  0001 C CNN
+F 0 "#PWR012" H 3840 2850 50  0001 C CNN
 F 1 "GND" H 3845 2927 50  0000 C CNN
 F 2 "" H 3840 3100 50  0001 C CNN
@@
 	7140 2645 7565 2645
 $Comp
-L Device:D_Schottky D?
+L Device:D_Schottky D1
 U 1 1 5DF67867
 P 7715 2645
-F 0 "D?" H 7715 2429 50  0000 C CNN
+F 0 "D1" H 7715 2429 50  0000 C CNN
 F 1 "D_Schottky" H 7715 2520 50  0000 C CNN
 F 2 "" H 7715 2645 50  0001 C CNN
@@
 5V_OUT
 $Comp
-L Jumper:SolderJumper_2_Open JP?
+L Jumper:SolderJumper_2_Open JP1
 U 1 1 5DF6A516
 P 4495 2995
-F 0 "JP?" V 4449 3063 50  0000 L CNN
+F 0 "JP1" V 4449 3063 50  0000 L CNN
 F 1 "boost_disable" V 4540 3063 50  0000 L CNN
 F 2 "" H 4495 2995 50  0001 C CNN
@@
 $EndComp
 $Comp
-L power:GND #PWR?
+L power:GND #PWR013
 U 1 1 5DF6A5BE
 P 4495 3425
-F 0 "#PWR?" H 4495 3175 50  0001 C CNN
+F 0 "#PWR013" H 4495 3175 50  0001 C CNN
 F 1 "GND" H 4500 3252 50  0000 C CNN
 F 2 "" H 4495 3425 50  0001 C CNN
@@
 	4495 3145 4495 3425
 $Comp
-L Device:D_Schottky D?
+L Device:D_Schottky D2
 U 1 1 5DF7CB12
 P 7720 2940
-F 0 "D?" H 7720 2724 50  0000 C CNN
+F 0 "D2" H 7720 2724 50  0000 C CNN
 F 1 "D_Schottky" H 7720 2815 50  0000 C CNN
 F 2 "" H 7720 2940 50  0001 C CNN

Commit message: Initial attempt at PCB
Signed-off-by: Tisham Dhar <whatnickd@gmail.com>
Parts:
- C1, C2, C3: footprint (none) -> Capacitor_SMD:C_0805_2012Metric
- D1, D2: footprint (none) -> Diode_SMD:D_SMB
- JP1: footprint (none) -> Jumper:SolderJumper-2_P1.3mm_Open_TrianglePad1.0x1.5mm
- L1: footprint (none) -> Inductor_SMD:L_6.3x6.3_H3
- R1, R2, R3: footprint (none) -> Resistor_SMD:R_0603_1608Metric
- U1: footprint SOP65P490X110-8N -> Package_SO:MSOP-8_3x3mm_P0.65mm
Changed lines of the file:
@@
 F 0 "U1" H 5605 4115 50  0000 C CNN
 F 1 "PAM2401SCADJ" H 5605 4024 50  0000 C CNN
-F 2 "SOP65P490X110-8N" H 5605 3245 50  0001 L BNN
+F 2 "Package_SO:MSOP-8_3x3mm_P0.65mm" H 5605 3245 50  0001 L BNN
 F 3 "Diodes Inc." H 5605 3245 50  0001 L BNN
 F 4 "Unavailable" H 5605 3245 50  0001 L BNN "Field4"
@@
 F 0 "L1" H 4039 2674 50  0000 R CNN
 F 1 "2.2uH/3A" H 4039 2765 50  0000 R CNN
-F 2 "" H 4080 2720 50  0001 C CNN
+F 2 "Inductor_SMD:L_6.3x6.3_H3" H 4080 2720 50  0001 C CNN
 F 3 "~" H 4080 2720 50  0001 C CNN
 	1    4080 2720
@@
 F 0 "C1" H 3932 2891 50  0000 L CNN
 F 1 "22u" H 3932 2800 50  0000 L CNN
-F 2 "" H 3840 2845 50  0001 C CNN
+F 2 "Capacitor_SMD:C_0805_2012Metric" H 3840 2845 50  0001 C CNN
 F 3 "~" H 3840 2845 50  0001 C CNN
 	1    3840 2845
@@
 F 0 "R3" H 6549 3366 50  0000 L CNN
 F 1 "100k" H 6549 3275 50  0000 L CNN
-F 2 "" H 6490 3320 50  0001 C CNN
+F 2 "Resistor_SMD:R_0603_1608Metric" H 6490 3320 50  0001 C CNN
 F 3 "~" H 6490 3320 50  0001 C CNN
 	1    6490 3320
@@
 F 0 "R2" H 6549 2971 50  0000 L CNN
 F 1 "750k" H 6549 2880 50  0000 L CNN
-F 2 "" H 6490 2925 50  0001 C CNN
+F 2 "Resistor_SMD:R_0603_1608Metric" H 6490 2925 50  0001 C CNN
 F 3 "~" H 6490 2925 50  0001 C CNN
 	1    6490 2925
@@
 F 0 "C3" H 7232 2961 50  0000 L CNN
 F 1 "22u" H 7232 2870 50  0000 L CNN
-F 2 "" H 7140 2915 50  0001 C CNN
+F 2 "Capacitor_SMD:C_0805_2012Metric" H 7140 2915 50  0001 C CNN
 F 3 "~" H 7140 2915 50  0001 C CNN
 	1    7140 2915
@@
 F 0 "C2" H 6997 2961 50  0000 L CNN
 F 1 "22u" H 6997 2870 50  0000 L CNN
-F 2 "" H 6905 2915 50  0001 C CNN
+F 2 "Capacitor_SMD:C_0805_2012Metric" H 6905 2915 50  0001 C CNN
 F 3 "~" H 6905 2915 50  0001 C CNN
 	1    6905 2915
@@
 F 0 "R1" H 4554 2746 50  0000 L CNN
 F 1 "10k" H 4554 2655 50  0000 L CNN
-F 2 "" H 4495 2700 50  0001 C CNN
+F 2 "Resistor_SMD:R_0603_1608Metric" H 4495 2700 50  0001 C CNN
 F 3 "~" H 4495 2700 50  0001 C CNN
 	1    4495 2700
@@
 F 0 "D1" H 7715 2429 50  0000 C CNN
 F 1 "D_Schottky" H 7715 2520 50  0000 C CNN
-F 2 "" H 7715 2645 50  0001 C CNN
+F 2 "Diode_SMD:D_SMB" H 7715 2645 50  0001 C CNN
 F 3 "~" H 7715 2645 50  0001 C CNN
 	1    7715 2645
@@
 F 0 "JP1" V 4449 3063 50  0000 L CNN
 F 1 "boost_disable" V 4540 3063 50  0000 L CNN
-F 2 "" H 4495 2995 50  0001 C CNN
+F 2 "Jumper:SolderJumper-2_P1.3mm_Open_TrianglePad1.0x1.5mm" H 4495 2995 50  0001 C CNN
 F 3 "~" H 4495 2995 50  0001 C CNN
 	1    4495 2995
@@
 F 0 "D2" H 7720 2724 50  0000 C CNN
 F 1 "D_Schottky" H 7720 2815 50  0000 C CNN
-F 2 "" H 7720 2940 50  0001 C CNN
+F 2 "Diode_SMD:D_SMB" H 7720 2940 50  0001 C CNN
 F 3 "~" H 7720 2940 50  0001 C CNN
 	1    7720 2940

Commit message: Initial cut at part placement
Signed-off-by: Tisham Dhar <whatnickd@gmail.com>
Parts:
- L1: footprint Inductor_SMD:L_6.3x6.3_H3 -> Inductor_SMD:L_Bourns-SRR1005
Changed lines of the file:
@@
 F 0 "L1" H 4039 2674 50  0000 R CNN
 F 1 "2.2uH/3A" H 4039 2765 50  0000 R CNN
-F 2 "Inductor_SMD:L_6.3x6.3_H3" H 4080 2720 50  0001 C CNN
+F 2 "Inductor_SMD:L_Bourns-SRR1005" H 4080 2720 50  0001 C CNN
 F 3 "~" H 4080 2720 50  0001 C CNN
 	1    4080 2720

Commit message: Note Inductor parts choice
Signed-off-by: Tisham Dhar <whatnickd@gmail.com>
Parts:
- L1: manf# (none) -> SRR1005-2R2M
Changed lines of the file:
@@
 F 1 "2.2uH/3A" H 4039 2765 50  0000 R CNN
 F 2 "Inductor_SMD:L_Bourns-SRR1005" H 4080 2720 50  0001 C CNN
-F 3 "~" H 4080 2720 50  0001 C CNN
+F 3 "https://www.bourns.com/docs/Product-Datasheets/SRR1005.pdf" H 4080 2720 50  0001 C CNN
+F 4 "SRR1005-2R2M" H 4080 2720 50  0001 C CNN "manf#"
 	1    4080 2720
 	-1   0    0    1
