File: Tph_Synth_Featherwing/boost_converter.sch (KiCad schematic (older format))
At the start: 11 parts, among them U1 PAM2401SCADJ

Commit message: More don't trust the autorouter
Signed-off-by: Tisham Dhar <whatnickd@gmail.com>
Connections:
- net BOOST_5V: now reaches C2.1, C3.1, D1.2 (A), R2.1, U1.7 (OUT)
Changed lines of the file:
@@
 Wire Wire Line
 	8005 2645 8175 2645
+Text Label 7235 2645 0    50   ~ 0
+BOOST_5V
 $EndSCHEMATC

Commit message: Added BOM and upgraded to kicad 5.0
Signed-off-by: Tisham Dhar <whatnickd@gmail.com>
Parts:
- C1, C2, C3: manf# (none) -> C2012JB1V226M125AC
- D1, D2: manf# (none) -> B330B-13-F
- JP1: DNP (none) -> (none)
- R1: manf# (none) -> RT0603FRD0710KL
- R2: manf# (none) -> RC0603FR-07750KL
- R3: manf# (none) -> RC0603FR-07100KL
- U1: manf# (none) -> PAM2401SCADJ
Changed lines of the file:
@@
 EESchema Schematic File Version 4
-LIBS:Tph_Synth_Featherwing-cache
-EELAYER 26 0
+EELAYER 30 0
 EELAYER END
 $Descr A4 11693 8268
@@
 F 7 "MSOP-8 Diodes Inc." H 5605 3245 50  0001 L BNN "Field7"
 F 8 "Conv DC-DC Single Step Up 0.9V to 4.75V 8-Pin MSOP T/R" H 5605 3245 50  0001 L BNN "Field8"
+F 9 "PAM2401SCADJ" H 5605 3245 50  0001 C CNN "manf#"
 	1    5605 3245
 	1    0    0    -1
@@
 F 2 "Capacitor_SMD:C_0805_2012Metric" H 3840 2845 50  0001 C CNN
 F 3 "~" H 3840 2845 50  0001 C CNN
+F 4 "C2012JB1V226M125AC" H 3840 2845 50  0001 C CNN "manf#"
 	1    3840 2845
 	1    0    0    -1
@@
 F 2 "Resistor_SMD:R_0603_1608Metric" H 6490 3320 50  0001 C CNN
 F 3 "~" H 6490 3320 50  0001 C CNN
+F 4 "RC0603FR-07100KL" H 6490 3320 50  0001 C CNN "manf#"
 	1    6490 3320
 	1    0    0    -1
@@
 F 2 "Resistor_SMD:R_0603_1608Metric" H 6490 2925 50  0001 C CNN
 F 3 "~" H 6490 2925 50  0001 C CNN
+F 4 "RC0603FR-07750KL" H 6490 2925 50  0001 C CNN "manf#"
 	1    6490 2925
 	1    0    0    -1
@@
 F 2 "Capacitor_SMD:C_0805_2012Metric" H 7140 2915 50  0001 C CNN
 F 3 "~" H 7140 2915 50  0001 C CNN
+F 4 "C2012JB1V226M125AC" H 7140 2915 50  0001 C CNN "manf#"
 	1    7140 2915
 	1    0    0    -1
@@
 F 2 "Capacitor_SMD:C_0805_2012Metric" H 6905 2915 50  0001 C CNN
 F 3 "~" H 6905 2915 50  0001 C CNN
+F 4 "C2012JB1V226M125AC" H 6905 2915 50  0001 C CNN "manf#"
 	1    6905 2915
 	1    0    0    -1
@@
 F 2 "Resistor_SMD:R_0603_1608Metric" H 4495 2700 50  0001 C CNN
 F 3 "~" H 4495 2700 50  0001 C CNN
+F 4 "RT0603FRD0710KL" H 4495 2700 50  0001 C CNN "manf#"
 	1    4495 2700
 	1    0    0    -1
@@
 F 2 "Diode_SMD:D_SMB" H 7715 2645 50  0001 C CNN
 F 3 "~" H 7715 2645 50  0001 C CNN
+F 4 "B330B-13-F" H 7715 2645 50  0001 C CNN "manf#"
 	1    7715 2645
 	-1   0    0    1
@@
 F 2 "Jumper:SolderJumper-2_P1.3mm_Open_TrianglePad1.0x1.5mm" H 4495 2995 50  0001 C CNN
 F 3 "~" H 4495 2995 50  0001 C CNN
+F 4 " " H 4495 2995 50  0001 C CNN "DNP"
 	1    4495 2995
 	0    1    1    0
@@
 F 2 "Diode_SMD:D_SMB" H 7720 2940 50  0001 C CNN
 F 3 "~" H 7720 2940 50  0001 C CNN
+F 4 "B330B-13-F" H 7720 2940 50  0001 C CNN "manf#"
 	1    7720 2940
 	-1   0    0    1
