File: Tph_Synth_Featherwing/quad_opamp_gain.sch (KiCad schematic (older format))
At the start: 26 parts, among them U3 Opamp_Quad_Generic

Commit message: Added BOM and upgraded to kicad 5.0
Signed-off-by: Tisham Dhar <whatnickd@gmail.com>
Parts:
- C10, C11, C18, C6, C7, C8, C9: manf# (none) -> GMK212BBJ106MG-T
- C12: manf# (none) -> GJM0335C1E5R0BB01D
- JP2, TP3, TP4, TP5: DNP (none) -> (none)
- R10: manf# (none) -> PV36W202C01B00
- R11, R12, R13, R14: manf# (none) -> RT0603CRE07100KL
- R15: manf# (none) -> CRT0603-FY-1001ELF
- R4, R5, R6: manf# (none) -> RT0603FRD0710KL
- R7, R8, R9, RV1: manf# (none) -> PTV09A-2020F-B104
- U3: manf# (none) -> LM324PWR
Changed lines of the file:
@@
 EESchema Schematic File Version 4
-LIBS:Tph_Synth_Featherwing-cache
-EELAYER 26 0
+EELAYER 30 0
 EELAYER END
 $Descr A4 11693 8268
@@
 F 2 "Package_SO:TSSOP-14_4.4x5mm_P0.65mm" H 2495 1295 50  0001 C CNN
 F 3 "~" H 2495 1295 50  0001 C CNN
+F 4 "LM324PWR" H 2495 1295 50  0001 C CNN "manf#"
 	1    2495 1295
 	1    0    0    -1
@@
 F 2 "Package_SO:TSSOP-14_4.4x5mm_P0.65mm" H 2520 2430 50  0001 C CNN
 F 3 "~" H 2520 2430 50  0001 C CNN
+F 4 "LM324PWR" H 2520 2430 50  0001 C CNN "manf#"
 	2    2520 2430
 	1    0    0    -1
@@
 F 2 "Package_SO:TSSOP-14_4.4x5mm_P0.65mm" H 2505 3455 50  0001 C CNN
 F 3 "~" H 2505 3455 50  0001 C CNN
+F 4 "LM324PWR" H 2505 3455 50  0001 C CNN "manf#"
 	3    2505 3455
 	1    0    0    -1
@@
 F 2 "Package_SO:TSSOP-14_4.4x5mm_P0.65mm" H 6930 1520 50  0001 C CNN
 F 3 "~" H 6930 1520 50  0001 C CNN
+F 4 "LM324PWR" H 6930 1520 50  0001 C CNN "manf#"
 	4    6930 1520
 	1    0    0    1
@@
 F 2 "Package_SO:TSSOP-14_4.4x5mm_P0.65mm" H 9835 1575 50  0001 C CNN
 F 3 "~" H 9835 1575 50  0001 C CNN
+F 4 "LM324PWR" H 9835 1575 50  0001 C CNN "manf#"
 	5    9835 1575
 	1    0    0    -1
@@
 F 2 "Resistor_SMD:R_0603_1608Metric" H 2095 1395 50  0001 C CNN
 F 3 "~" H 2095 1395 50  0001 C CNN
+F 4 "RT0603FRD0710KL" H 2095 1395 50  0001 C CNN "manf#"
 	1    2095 1395
 	0    1    1    0
@@
 F 2 "Resistor_SMD:R_0603_1608Metric" H 2120 2530 50  0001 C CNN
 F 3 "~" H 2120 2530 50  0001 C CNN
+F 4 "RT0603FRD0710KL" H 2120 2530 50  0001 C CNN "manf#"
 	1    2120 2530
 	0    1    1    0
@@
 F 2 "Resistor_SMD:R_0603_1608Metric" H 2105 3555 50  0001 C CNN
 F 3 "~" H 2105 3555 50  0001 C CNN
+F 4 "RT0603FRD0710KL" H 2105 3555 50  0001 C CNN "manf#"
 	1    2105 3555
 	0    1    1    0
@@
 F 2 "Resistor_SMD:R_0603_1608Metric" H 6880 2005 50  0001 C CNN
 F 3 "~" H 6880 2005 50  0001 C CNN
+F 4 "RT0603CRE07100KL" H 6880 2005 50  0001 C CNN "manf#"
 	1    6880 2005
 	0    1    1    0
@@
 F 2 "Potentiometer_THT:Potentiometer_Bourns_PTV09A-2_Single_Horizontal" V 2385 1645 50  0001 C CNN
 F 3 "~" H 2455 1645 50  0001 C CNN
+F 4 "PTV09A-2020F-B104" H 2455 1645 50  0001 C CNN "manf#"
 	1    2455 1645
 	0    1    1    0
@@
 F 2 "Potentiometer_THT:Potentiometer_Bourns_PTV09A-2_Single_Horizontal" V 2385 2765 50  0001 C CNN
 F 3 "~" H 2455 2765 50  0001 C CNN
+F 4 "PTV09A-2020F-B104" H 2455 2765 50  0001 C CNN "manf#"
 	1    2455 2765
 	0    1    1    0
@@
 F 2 "Potentiometer_THT:Potentiometer_Bourns_PTV09A-2_Single_Horizontal" V 2365 3810 50  0001 C CNN
 F 3 "~" H 2435 3810 50  0001 C CNN
+F 4 "PTV09A-2020F-B104" H 2435 3810 50  0001 C CNN "manf#"
 	1    2435 3810
 	0    1    1    0
@@
 F 2 "Potentiometer_THT:Potentiometer_Bourns_3296W_Vertical" V 5990 2005 50  0001 C CNN
 F 3 "~" H 6060 2005 50  0001 C CNN
+F 4 "PV36W202C01B00" H 6060 2005 50  0001 C CNN "manf#"
 	1    6060 2005
 	0    -1   -1   0
@@
 F 2 "Capacitor_SMD:C_0805_2012Metric" H 1905 3555 50  0001 C CNN
 F 3 "~" H 1905 3555 50  0001 C CNN
+F 4 "GMK212BBJ106MG-T" H 1905 3555 50  0001 C CNN "manf#"
 	1    1905 3555
 	0    1    1    0
@@
 F 2 "Capacitor_SMD:C_0805_2012Metric" H 1920 2530 50  0001 C CNN
 F 3 "~" H 1920 2530 50  0001 C CNN
+F 4 "GMK212BBJ106MG-T" H 1920 2530 50  0001 C CNN "manf#"
 	1    1920 2530
 	0    1    1    0
@@
 F 2 "Capacitor_SMD:C_0805_2012Metric" H 1895 1395 50  0001 C CNN
 F 3 "~" H 1895 1395 50  0001 C CNN
+F 4 "GMK212BBJ106MG-T" H 1895 1395 50  0001 C CNN "manf#"
 	1    1895 1395
 	0    1    1    0
@@
 F 2 "Capacitor_SMD:C_0805_2012Metric" H 2895 1295 50  0001 C CNN
 F 3 "~" H 2895 1295 50  0001 C CNN
+F 4 "GMK212BBJ106MG-T" H 2895 1295 50  0001 C CNN "manf#"
 	1    2895 1295
 	0    1    1    0
@@
 F 2 "Capacitor_SMD:C_0805_2012Metric" H 2920 2430 50  0001 C CNN
 F 3 "~" H 2920 2430 50  0001 C CNN
+F 4 "GMK212BBJ106MG-T" H 2920 2430 50  0001 C CNN "manf#"
 	1    2920 2430
 	0    1    1    0
@@
 F 2 "Capacitor_SMD:C_0805_2012Metric" H 2905 3455 50  0001 C CNN
 F 3 "~" H 2905 3455 50  0001 C CNN
+F 4 "GMK212BBJ106MG-T" H 2905 3455 50  0001 C CNN "manf#"
 	1    2905 3455
 	0    1    1    0
@@
 F 2 "Resistor_SMD:R_0603_1608Metric" H 6900 1130 50  0001 C CNN
 F 3 "~" H 6900 1130 50  0001 C CNN
+F 4 "RT0603CRE07100KL" H 6900 1130 50  0001 C CNN "manf#"
 	1    6900 1130
 	0    1    1    0
@@
 F 2 "Resistor_SMD:R_0603_1608Metric" H 6310 1130 50  0001 C CNN
 F 3 "~" H 6310 1130 50  0001 C CNN
+F 4 "RT0603CRE07100KL" H 6310 1130 50  0001 C CNN "manf#"
 	1    6310 1130
 	0    1    1    0
@@
 F 2 "Capacitor_SMD:C_0603_1608Metric" H 6910 1265 50  0001 C CNN
 F 3 "~" H 6910 1265 50  0001 C CNN
+F 4 "GJM0335C1E5R0BB01D" H 6910 1265 50  0001 C CNN "manf#"
 	1    6910 1265
 	0    -1   -1   0
@@
 F 2 "Resistor_SMD:R_0603_1608Metric" H 7420 2005 50  0001 C CNN
 F 3 "~" H 7420 2005 50  0001 C CNN
+F 4 "CRT0603-FY-1001ELF" H 7420 2005 50  0001 C CNN "manf#"
 	1    7420 2005
 	0    1    1    0
@@
 F 2 "Resistor_SMD:R_0603_1608Metric" H 6420 2005 50  0001 C CNN
 F 3 "~" H 6420 2005 50  0001 C CNN
+F 4 "RT0603CRE07100KL" H 6420 2005 50  0001 C CNN "manf#"
 	1    6420 2005
 	0    1    1    0
@@
 F 2 "Potentiometer_THT:Potentiometer_Bourns_PTV09A-2_Single_Horizontal" H 5760 2005 50  0001 C CNN
 F 3 "~" H 5760 2005 50  0001 C CNN
+F 4 "PTV09A-2020F-B104" H 5760 2005 50  0001 C CNN "manf#"
 	1    5760 2005
 	1    0    0    -1
@@
 F 2 "TestPoint:TestPoint_Pad_D1.0mm" H 6830 2005 50  0001 C CNN
 F 3 "~" H 6830 2005 50  0001 C CNN
+F 4 " " H 6630 2005 50  0001 C CNN "DNP"
 	1    6630 2005
 	-1   0    0    1
@@
 F 2 "TestPoint:TestPoint_Pad_D1.0mm" H 7795 2005 50  0001 C CNN
 F 3 "~" H 7795 2005 50  0001 C CNN
+F 4 " " H 7595 2005 50  0001 C CNN "DNP"
 	1    7595 2005
 	0    1    1    0
@@
 F 2 "TestPoint:TestPoint_Pad_D1.0mm" H 6110 2005 50  0001 C CNN
 F 3 "~" H 6110 2005 50  0001 C CNN
+F 4 " " H 5910 2005 50  0001 C CNN "DNP"
 	1    5910 2005
 	1    0    0    -1
@@
 F 2 "Capacitor_SMD:C_0805_2012Metric" H 5760 1660 50  0001 C CNN
 F 3 "~" H 5760 1660 50  0001 C CNN
+F 4 "GMK212BBJ106MG-T" H 5760 1660 50  0001 C CNN "manf#"
 	1    5760 1660
 	1    0    0    -1
@@
 F 2 "Jumper:SolderJumper-2_P1.3mm_Open_TrianglePad1.0x1.5mm" H 5520 1615 50  0001 C CNN
 F 3 "~" H 5520 1615 50  0001 C CNN
+F 4 " " H 5520 1615 50  0001 C CNN "DNP"
 	1    5520 1615
 	0    -1   -1   0
